Commit message: RViz launch profiles (I15) and fix the MotionPlanning display
Adds the two supported RViz entry points and closes the MotionPlanning
display defect that had been documented as an open issue.

MotionPlanning fix
------------------
The display never loaded its robot model: loadRobotModel aborted with
InvalidParameterTypeException on a double-valued kinematics parameter,
leaving NO PLANNING LIBRARY LOADED and no interactive markers.

Root cause is the process locale, not the launch plumbing. rviz2's
main.cpp constructs QApplication before rclcpp::init, and QApplication
calls setlocale(LC_ALL, ""), so the process leaves the C locale that
every C program starts in. rcl_yaml_param_parser accepts a scalar as a
double only when strtod consumes it whole, so under a comma-decimal
LC_NUMERIC "0.005" is stored as a string. MoveIt's kinematics
ParamListener then declares that key as a statically typed double,
rclcpp rejects the string override, and RobotModelLoader - which
catches only ParameterTypeException - lets it escape.

This is why removing parameters only moved the failure: every double
reaching rviz2 was corrupt, so dropping joint_limits (max_velocity 0.75)
merely exposed the next one (kinematics_solver_search_resolution 0.005).
max_acceleration 2.0 never appeared because strtod does consume "2.0"
even in tr_TR. move_group was never affected because it has no Qt.

Fix: additional_env={"LC_NUMERIC": "C"} on the rviz2 node in
sim_moveit.launch.py. Applies to any comma-decimal locale, not just
Turkish. Also drops a redundant Move Group Namespace key from
moveit.rviz and adds a CI guard so the env pin cannot be removed
silently.

Verified under the real tr_TR shell: no loadRobotModel exception, the
kinematics parameter reads back as Double 0.005, /query_planner_interface
returns OMPL and RRTConnectkConfigDefault for all three groups, both
gripper markers drag via IK, and Plan & Execute drives both arm
controllers to SUCCEEDED in Gazebo. Bare headless launch still starts
with no RViz.

Also in this change
-------------------
- baxter_gz_sim: sim_rviz profile, checked-in sim.rviz and gz_gui.config,
  deterministic pedestal mount, all 17 independent joint states,
  controller command limits and finite tolerances.
- baxter_moveit_config: sim_moveit_rviz profile, moveit.rviz, a
  readiness gate replacing the arbitrary startup timer, and a sim-only
  move_group executable with clean teardown.
- baxter_examples: ik_service_client and moveit_pose clients; reversible,
  numerically checked motion examples.
- Docs and release metadata updated; known_issues.md records the defect,
  its root cause, and the correction to the earlier ruled-out verdict.

File: src/baxter_gz_sim/urdf/baxter_gz_control.urdf.xacro (robot description, xacro)
@@ -11,8 +11,24 @@
   <xacro:include filename="$(find baxter_description)/urdf/left_end_effector.urdf.xacro"/>
   <xacro:include filename="$(find baxter_description)/urdf/right_end_effector.urdf.xacro"/>
-  <xacro:macro name="arm_ros2_control_joint" params="joint_name">
+  <link name="world"/>
+  <joint name="world_joint" type="fixed">
+    <origin xyz="0 0 0.92418" rpy="0 0 0"/>
+    <parent link="world"/>
+    <child link="base"/>
+  </joint>
+  <xacro:macro name="arm_ros2_control_joint" params="joint_name initial_position">
     <joint name="${joint_name}">
       <command_interface name="position"/>
-      <state_interface name="position"/>
+      <state_interface name="position">
+        <param name="initial_value">${initial_position}</param>
+      </state_interface>
+      <state_interface name="velocity"/>
+    </joint>
+  </xacro:macro>
+  <xacro:macro name="state_only_ros2_control_joint" params="joint_name initial_position">
+    <joint name="${joint_name}">
+      <state_interface name="position">
+        <param name="initial_value">${initial_position}</param>
+      </state_interface>
       <state_interface name="velocity"/>
     </joint>
@@ -22,18 +38,21 @@
       <plugin>gz_ros2_control/GazeboSimSystem</plugin>
     </hardware>
-    <xacro:arm_ros2_control_joint joint_name="left_s0"/>
-    <xacro:arm_ros2_control_joint joint_name="left_s1"/>
-    <xacro:arm_ros2_control_joint joint_name="left_e0"/>
-    <xacro:arm_ros2_control_joint joint_name="left_e1"/>
-    <xacro:arm_ros2_control_joint joint_name="left_w0"/>
-    <xacro:arm_ros2_control_joint joint_name="left_w1"/>
-    <xacro:arm_ros2_control_joint joint_name="left_w2"/>
-    <xacro:arm_ros2_control_joint joint_name="right_s0"/>
-    <xacro:arm_ros2_control_joint joint_name="right_s1"/>
-    <xacro:arm_ros2_control_joint joint_name="right_e0"/>
-    <xacro:arm_ros2_control_joint joint_name="right_e1"/>
-    <xacro:arm_ros2_control_joint joint_name="right_w0"/>
-    <xacro:arm_ros2_control_joint joint_name="right_w1"/>
-    <xacro:arm_ros2_control_joint joint_name="right_w2"/>
+    <xacro:arm_ros2_control_joint joint_name="left_s0" initial_position="0.0"/>
+    <xacro:arm_ros2_control_joint joint_name="left_s1" initial_position="-0.55"/>
+    <xacro:arm_ros2_control_joint joint_name="left_e0" initial_position="0.0"/>
+    <xacro:arm_ros2_control_joint joint_name="left_e1" initial_position="0.75"/>
+    <xacro:arm_ros2_control_joint joint_name="left_w0" initial_position="0.0"/>
+    <xacro:arm_ros2_control_joint joint_name="left_w1" initial_position="1.26"/>
+    <xacro:arm_ros2_control_joint joint_name="left_w2" initial_position="0.0"/>
+    <xacro:arm_ros2_control_joint joint_name="right_s0" initial_position="0.0"/>
+    <xacro:arm_ros2_control_joint joint_name="right_s1" initial_position="-0.55"/>
+    <xacro:arm_ros2_control_joint joint_name="right_e0" initial_position="0.0"/>
+    <xacro:arm_ros2_control_joint joint_name="right_e1" initial_position="0.75"/>
+    <xacro:arm_ros2_control_joint joint_name="right_w0" initial_position="0.0"/>
+    <xacro:arm_ros2_control_joint joint_name="right_w1" initial_position="1.26"/>
+    <xacro:arm_ros2_control_joint joint_name="right_w2" initial_position="0.0"/>
+    <xacro:state_only_ros2_control_joint joint_name="head_pan" initial_position="0.0"/>
+    <xacro:state_only_ros2_control_joint joint_name="l_gripper_l_finger_joint" initial_position="0.0"/>
+    <xacro:state_only_ros2_control_joint joint_name="r_gripper_l_finger_joint" initial_position="0.0"/>
   </ros2_control>
   <gazebo>
